File: hardware/Matrix6/Matrix6.kicad_pcb (KiCad board)
At the start: 4 copper layers, 35.6 x 61 mm, 32 parts, among them J1 USB4105-GF-A-120, J2 GPIO / POWER, J3 GPIO / POWER, SW1 RESET, SW2 BOOT, U1 ESP32-S3-WROOM-1-N8R8, U2 AP63203WU-7, U3 USBLC6-2SC6

Commit message: Align Matrix6 v0.5 headers and manual routing with Matrix5 shields
Use two 20-pin sockets at 33.02 mm spacing and remap the GPIO and power nets against Matrix5 Main and all eleven shield designs. Document the three unused USB/VBAT pins, fused VBUS output and prototype power/mechanical limits.

Preserve the reviewed USB copper, connector body keepout, continuous L2 GND and design rules. Include schematic/PCB/3D previews and reproducible DRC, ERC, pin-map, keepout and electrical checks; all current DRC/ERC/parity/unconnected checks pass.
Parts:
- removed J2, J3: GPIO / POWER, Connector_PinHeader_2.54mm:PinHeader_1x20_P2.54mm_Vertical
- added H1: Matrix5 H1, Connector_PinSocket_2.54mm:PinSocket_1x20_P2.54mm_Vertical, F.Cu at (101.3, 153.3)
- added H2: Matrix5 H2, Connector_PinSocket_2.54mm:PinSocket_1x20_P2.54mm_Vertical, F.Cu at (134.3, 153.3)
Routing:
- net /IO1: track 11.1 -> 67.6 mm, vias 1 -> 3
- net /IO2: track 12.3 -> 63.8 mm, vias 1 -> 3
- net /IO17: track 18.7 -> 63.9 mm, vias 1 -> 3
- net /IO18: track 19.9 -> 58.2 mm, vias 1 -> 3
- net /+5V: track 59.7 -> 28.0 mm
- net /IO0: track 68.2 -> 95.9 mm, vias 3 -> 6
- net /IO4: track 11.1 -> 38.2 mm, vias 1 -> 2
- net /IO5: track 12.3 -> 34.4 mm, vias 1 -> 2
- net /IO11: track 37.4 -> 17.9 mm, vias 1 -> 2
- net /IO12: track 41.2 -> 22.4 mm, vias 1 -> 2
- net /IO10: track 33.6 -> 15.4 mm, vias 1 -> 2
- net /IO6: track 13.6 -> 30.6 mm, vias 1 -> 2
- net /IO9: track 29.8 -> 15.8 mm, vias 1 -> 2
- net /IO48: track 29.2 -> 43.0 mm, vias 1 -> 5
- net /IO7: track 14.9 -> 26.8 mm, vias 1 -> 2
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Other:
- board size 35.6 x 61 mm -> 40.6 x 61 mm
- board text added: "MATRIX6"
- board text added: "N8R8 v0.5"
- board text added: "NC"
- board text added: "VBUS"
- board text removed: "5V"
- board text removed: "N8R8 v0.4"
- board text removed: "S3 DEV"

Commit message: Add rear microSD with clear extraction path and LiPo power to Matrix Six
Parts:
- added C10: 22uF 25V X5R, Capacitor_SMD:C_0805_2012Metric, B.Cu at (129.7, 154.8)
- added C11: 22uF 25V X5R, Capacitor_SMD:C_0805_2012Metric, B.Cu at (105.8, 141.2)
- added C12: 100nF, Capacitor_SMD:C_0603_1608Metric, B.Cu at (117.3, 142.4)
- added C9: 22uF 25V X5R, Capacitor_SMD:C_0805_2012Metric, B.Cu at (129.5, 151.6)
- added J2: microSD (rear), Connector_Card:microSD_HC_Hirose_DM3AT-SF-PEJM5, B.Cu at (117.8, 132.0)
- added J3: LiPo 1S / PH2, Connector_JST:JST_PH_S2B-PH-K_1x02_P2.00mm_Horizontal, B.Cu at (108.5, 153.5)
- added Q1: AO3401A, Package_TO_SOT_SMD:SOT-23, B.Cu at (123.0, 146.0)
- added R12: 100R, Resistor_SMD:R_0603_1608Metric, F.Cu at (125.7, 140.0)
- added R13: 10k / 100mA, Resistor_SMD:R_0603_1608Metric, B.Cu at (128.5, 143.5)
- added R14: 100k, Resistor_SMD:R_0603_1608Metric, B.Cu at (130.5, 142.5)
- added R15: 10k, Resistor_SMD:R_0603_1608Metric, B.Cu at (120.6, 142.7)
- added R16: 10k, Resistor_SMD:R_0603_1608Metric, F.Cu at (113.0, 128.0)
- added R17: 10k, Resistor_SMD:R_0603_1608Metric, F.Cu at (115.0, 128.0)
- added R18: 10k, Resistor_SMD:R_0603_1608Metric, F.Cu at (117.0, 128.0)
- added R19: 10k, Resistor_SMD:R_0603_1608Metric, F.Cu at (117.5, 130.4)
- added U4: MCP73831 / 100mA, Package_TO_SOT_SMD:SOT-23-5, B.Cu at (128.5, 147.0)
- C1: value 22uF 16V X5R -> 22uF 25V X5R
- C2, C8: value 22uF 10V X5R -> 22uF 25V X5R
- C7: value 100nF 16V X7R -> 100nF
- L1: value 4.7uH SRN4018-4R7M -> 2.2uH / 3A
- R7: value 10k 1% -> 10k
- U2: value AP63203WU-7 -> TPS63001 (3.3V); footprint Package_TO_SOT_SMD:TSOT-23-6 -> Package_SON:Texas_DRC0010J
- moved C2 9.92 mm to (118.6, 132.8), turned to 0 degrees
- moved C7 6.49 mm to (125.3, 135.4)
- moved L1 5.40 mm to (116.9, 138.0), turned to 90 degrees
- moved U2 4.00 mm to (121.5, 138.0)
- moved C1 3.04 mm to (120.4, 142.2), turned to 180 degrees
- moved C8 1.06 mm to (121.5, 144.8), turned to 0 degrees
- moved R7 0.85 mm to (122.0, 128.8), turned to 90 degrees
Connections:
- C1 pad 1: /+5V -> /VSYS
- C7 pad 1: /BUCK_BST -> /VINA
- C7 pad 2: /BUCK_SW -> /GND
- D1 pad 1: /+5V -> /VSYS
- H2 pad 20: unconnected-(H2-Pin_20-Pad20) -> /VBAT
- L1 pad 1: /BUCK_SW -> /SW_L1
- L1 pad 2: /+3V3 -> /SW_L2
- U2 pad 2: /+5V -> /SW_L2
- U2 pad 3: /+5V -> /GND
- U2 pad 4: /GND -> /SW_L1
- U2 pad 5: /BUCK_SW -> /VSYS
- U2 pad 6: /BUCK_BST -> /VSYS
Routing:
- net /VBAT: track 0.00 -> 100.8 mm, vias 0 -> 4
- net /IO11: track 17.9 -> 80.0 mm, vias 2 -> 4
- net /IO13: track 26.1 -> 83.9 mm, vias 2 -> 4
- net /IO10: track 15.4 -> 66.8 mm, vias 2 -> 7
- net /IO12: track 22.4 -> 70.4 mm, vias 2 -> 3
- net /VSYS: track 0.00 -> 33.3 mm, vias 0 -> 4
- net /+5V: track 28.0 -> 0.00 mm, vias 4 -> 0
- net /+3V3: track 180.9 -> 203.5 mm, vias 6 -> 10
- net /VBUS_FUSED: track 32.7 -> 53.7 mm, vias 1 -> 4
- net /SD_DAT1: track 0.00 -> 12.8 mm, vias 0 -> 1
- net /IO0: track 95.9 -> 105.3 mm, vias 6 -> 4
- net /GND: track 14.4 -> 21.7 mm, vias 29 -> 33
- net /VINA: track 0.00 -> 6.58 mm
- net /IO48: track 43.0 -> 49.4 mm, vias 5 -> 2
- net /BUCK_SW: track 5.84 -> 0.00 mm
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Other:
- board text added: "+"
- board text added: "-"
- board text added: "BAT"
- board text added: "LiPo 1S"
- board text added: "Matrix Six"
- board text added: "microSD"
- board text removed: "3V3 GPIO ONLY"
- board text removed: "ESP32-S3"
- board text removed: "MATRIX6"
- board text removed: "N8R8 / USB-JTAG"
- board text removed: "N8R8 v0.5"
